Commit message: Model correctly inserted into gazebo, sensor plugins added.

File: pulsar_description/urdf/pulsar.urdf.xacro (robot description, xacro)
@@ -4,7 +4,16 @@
 <xacro:include filename="$(find pulsar_description)/urdf/chassis/chassis.urdf.xacro"/>
 <xacro:include filename="$(find pulsar_description)/urdf/wheel/wheel.urdf.xacro"/>
+<xacro:include filename="$(find pulsar_description)/urdf/laser_range_finder/laser_range_finder.urdf.xacro"/>
+<xacro:include filename="$(find pulsar_description)/urdf/imu/imu.urdf.xacro"/>
 <link name="base_link"/>
+<gazebo>
+    <self_collide>false</self_collide>
+</gazebo>
 <xacro:chassis/>
-<xacro:wheel name="left" y_pos="0.02"/>
-<xacro:wheel name="right" y_pos="-0.02"/>
+<xacro:wheel name="left" side="1"/>
+<xacro:wheel name="right" side="-1"/>
+<xacro:laser_range_finder name="left_range_finder" yaw="0.5236"/>
+<xacro:laser_range_finder name="middle_range_finder" yaw="0.0"/>
+<xacro:laser_range_finder name="right_range_finder" yaw="-0.5236"/>
+<xacro:imu/>
 </robot>

File: pulsar_description/urdf/wheel/wheel.urdf.xacro (robot description, xacro)
@@ -1,11 +1,11 @@
 <?xml version="1.0"?>
 <robot xmlns:xacro="http://www.ros.org/wiki/xacro">
-<xacro:macro name="wheel" params="y_pos name">
+<xacro:macro name="wheel" params="side name">
     <link name="${name}_wheel_link">
         <visual name="${name}_wheel_visual">
-            <origin xyz="0 0 0" rpy="1.57 0 0"/>
+            <origin xyz="-0.015 ${side*0.015} -0.015" rpy="1.57 0 0"/>
             <geometry>
                 <mesh filename="$(find pulsar_description)/meshes/wheel.stl"
-                      scale="0.001 0.001 0.001"/>
+                      scale="0.001 0.001 ${side*0.001}"/>
             </geometry>
         </visual>
@@ -16,16 +16,16 @@
             </geometry>
         </collision>
-        <inertia>
+        <inertial>
             <origin xyz="0 0 0" rpy="0 0 0"/>
             <mass value="0.005"/>
             <inertia ixx="2.879e-7" ixy="0.0" ixz="0.0"
                      iyy="5.625e-7" iyz="0.0" izz="2.879e-7"/>
-        </inertia>
+        </inertial>
     </link>
     <joint name="${name}_wheel_joint" type="continuous">
-        <origin xyz="0 ${y_pos} 0.015" rpy="0 0 0"/>
+        <origin xyz="0 ${side*0.02} 0.015" rpy="0 0 0"/>
         <limit effort="0.02" velocity="12"/>
-        <axis xyz="0 1 0"/>
-        <parent link="base_link"/>
+        <axis xyz="0 1 0" rpy="0 0 0"/>
+        <parent link="chassis"/>
         <child link="${name}_wheel_link"/>
     </joint>

Commit message: Successfully got robot moving in simulation. Need to tune PI values before beginning to look at kalman filter results.

File: pulsar_description/urdf/pulsar.urdf.xacro (robot description, xacro)
@@ -22,7 +22,7 @@
         <Q_th_dot>1e-6</Q_th_dot>
         <!-- Motor controller parameters -->
-        <motorKp>20</motorKp>
+        <motorKp>0.07</motorKp>
         <motorKi>0</motorKi>
-        <motorMaxTorque>1</motorMaxTorque>
+        <motorMaxTorque>0.006</motorMaxTorque>
         <!-- Odometry parameters -->
         <cpr>4000</cpr>

File: pulsar_description/urdf/wheel/wheel.urdf.xacro (robot description, xacro)
@@ -25,5 +25,6 @@
     <joint name="${name}_wheel_joint" type="continuous">
         <origin xyz="0 ${side*0.02} 0.015" rpy="0 0 0"/>
-        <limit effort="0.02" velocity="12"/>
+        <limit effort="0.006" velocity="7"/>
+        <dynamics damping="${0.5*0.006/7}" friction="0.0"/>
         <axis xyz="0 1 0" rpy="0 0 0"/>
         <parent link="chassis"/>
