Commit message: Some progress being made to tuning motor controllers for the simulation - not complete yet however.

File: pulsar_description/urdf/chassis/chassis.urdf.xacro (robot description, xacro)
@@ -35,5 +35,5 @@
         </collision>
         <inertial>
-            <origin xyz="-0.015 0 0.02" rpy="0 0 0"/>
+            <origin xyz="-0.01 0 0.02" rpy="0 0 0"/>
             <mass value="0.05"/>
             <inertia ixx="1.042e-5" ixy="0.0" ixz="0.0"
@@ -45,4 +45,9 @@
         <child link="chassis"/>
     </joint>
+    <gazebo reference="chassis">
+        <mu>0.2</mu>
+        <mu2>0.2</mu2>
+        <min_depth>0.003</min_depth>
+    </gazebo>
 </xacro:macro>
 </robot>

File: pulsar_description/urdf/pulsar.urdf.xacro (robot description, xacro)
@@ -22,12 +22,13 @@
         <Q_th_dot>1e-6</Q_th_dot>
         <!-- Motor controller parameters -->
-        <motorKp>0.07</motorKp>
-        <motorKi>0</motorKi>
+        <motorKp>0.09</motorKp>
+        <motorKi>0.0</motorKi>
+        <!--<motorMaxTorque>0.006</motorMaxTorque>-->
         <motorMaxTorque>0.006</motorMaxTorque>
         <!-- Odometry parameters -->
         <cpr>4000</cpr>
         <wheelRadius>0.015</wheelRadius>
-        <wheelSeparation>0.02</wheelSeparation>
-        <updateRate>10</updateRate>
+        <wheelSeparation>0.0375</wheelSeparation>
+        <updateRate>100</updateRate>
         <odomUniformNoise>0.01</odomUniformNoise>
         <!-- Wheel joints -->

File: pulsar_description/urdf/wheel/wheel.urdf.xacro (robot description, xacro)
@@ -4,5 +4,5 @@
     <link name="${name}_wheel_link">
         <visual name="${name}_wheel_visual">
-            <origin xyz="-0.015 ${side*0.015} -0.015" rpy="1.57 0 0"/>
+            <origin xyz="-0.0155 ${side*0.015} -0.0155" rpy="1.57 0 0"/>
             <geometry>
                 <mesh filename="$(find pulsar_description)/meshes/wheel.stl"
@@ -26,9 +26,14 @@
         <origin xyz="0 ${side*0.02} 0.015" rpy="0 0 0"/>
         <limit effort="0.006" velocity="7"/>
-        <dynamics damping="${0.5*0.006/7}" friction="0.0"/>
+        <dynamics damping="${0.25*0.006/7}" friction="0.0"/>
         <axis xyz="0 1 0" rpy="0 0 0"/>
         <parent link="chassis"/>
         <child link="${name}_wheel_link"/>
     </joint>
+    <gazebo reference="${name}_wheel_link">
+        <mu>1000</mu>
+        <mu2>1000</mu2>
+        <min_depth>0.002</min_depth>
+    </gazebo>
 </xacro:macro>
 </robot>

Commit message: Relatively tuned motor PI controller for simulation
Kalman filter spits out NaN values so that needs to be fixed next.

File: pulsar_description/urdf/chassis/chassis.urdf.xacro (robot description, xacro)
@@ -23,5 +23,5 @@
         </collision>
         <collision name="front_caster_collision">
-            <origin xyz="0.02 0 0.003" rpy="0 0 0"/>
+            <origin xyz="0.02 0 0.004" rpy="0 0 0"/>
             <geometry>
                 <sphere radius="0.003"/>
@@ -29,5 +29,5 @@
         </collision>
         <collision name="rear_caster_collision">
-            <origin xyz="-0.025 0 0.003" rpy="0 0 0"/>
+            <origin xyz="-0.025 0 0.004" rpy="0 0 0"/>
             <geometry>
                 <sphere radius="0.003"/>
@@ -46,7 +46,7 @@
     </joint>
     <gazebo reference="chassis">
-        <mu>0.2</mu>
-        <mu2>0.2</mu2>
-        <min_depth>0.003</min_depth>
+        <mu>0.02</mu>
+        <mu2>0.02</mu2>
+        <min_depth>0.002</min_depth>
     </gazebo>
 </xacro:macro>

File: pulsar_description/urdf/pulsar.urdf.xacro (robot description, xacro)
@@ -22,6 +22,6 @@
         <Q_th_dot>1e-6</Q_th_dot>
         <!-- Motor controller parameters -->
-        <motorKp>0.09</motorKp>
-        <motorKi>0.0</motorKi>
+        <motorKp>0.08</motorKp>
+        <motorKi>0.8</motorKi>
         <!--<motorMaxTorque>0.006</motorMaxTorque>-->
         <motorMaxTorque>0.006</motorMaxTorque>

File: pulsar_description/urdf/wheel/wheel.urdf.xacro (robot description, xacro)
@@ -26,5 +26,5 @@
         <origin xyz="0 ${side*0.02} 0.015" rpy="0 0 0"/>
         <limit effort="0.006" velocity="7"/>
-        <dynamics damping="${0.25*0.006/7}" friction="0.0"/>
+        <dynamics damping="${0.25*0.006/7}" friction="0.0006"/>
         <axis xyz="0 1 0" rpy="0 0 0"/>
         <parent link="chassis"/>
