Commit message: Some mods to range finder coning. Updated world to have walls.

File: pulsar_description/urdf/laser_range_finder/laser_range_finder.urdf.xacro (robot description, xacro)
@@ -1,5 +1,5 @@
 <?xml version="1.0"?>
 <robot xmlns:xacro="http://www.ros.org/wiki/xacro">
-<xacro:property name="cone_angle" value="0.26"/>
+<xacro:property name="cone_angle" value="0.09"/>
 <xacro:property name="update_rate" value="10"/>
 <xacro:macro name="laser_range_finder" params="name yaw">
@@ -28,4 +28,5 @@
         <sensor type="ray" name="${name}_sensor">
             <pose>0 0 0 0 0 0</pose>
+            <visualize>true</visualize>
             <update_rate>${update_rate}</update_rate>
             <ray>
